Commit message: upgrade Robbie 5 to robbie 7

File: urdf/robbie7.xacro (robot description, xacro)
@@ -32,5 +32,5 @@
    <visual>
       <geometry>
-        <mesh filename="package://robbie/meshes/upper_torso2.stl" scale="${M_SCALE} ${M_SCALE} ${M_SCALE}"/>
+        <mesh filename="package://robbie/mesh/upper_torso2.stl" scale="${M_SCALE} ${M_SCALE} ${M_SCALE}"/>
       </geometry>
          <material name="green">
@@ -43,5 +43,5 @@
    <visual>
       <geometry>
-        <mesh filename="package://robbie/meshes/bottom torso.stl" scale="${M_SCALE} ${M_SCALE} ${M_SCALE}"/>
+        <mesh filename="package://robbie/mesh/bottom torso.stl" scale="${M_SCALE} ${M_SCALE} ${M_SCALE}"/>
       </geometry>
           <xacro:cyan3 />
@@ -52,5 +52,5 @@
    <visual>
       <geometry>
-        <mesh filename="package://robbie/meshes/waist top lower left.stl" scale="${M_SCALE} ${M_SCALE} ${M_SCALE}"/>
+        <mesh filename="package://robbie/mesh/waist top lower left.stl" scale="${M_SCALE} ${M_SCALE} ${M_SCALE}"/>
       </geometry>
           <xacro:cyan3 />
@@ -61,5 +61,5 @@
    <visual>
       <geometry>
-        <mesh filename="package://robbie/meshes/waist top lower right.stl" scale="${M_SCALE} ${M_SCALE} ${M_SCALE}"/>
+        <mesh filename="package://robbie/mesh/waist top lower right.stl" scale="${M_SCALE} ${M_SCALE} ${M_SCALE}"/>
       </geometry>
           <xacro:cyan3 />
@@ -70,5 +70,5 @@
    <visual>
       <geometry>
-        <mesh filename="package://robbie/meshes/waist top upper left.stl" scale="${M_SCALE} ${M_SCALE} ${M_SCALE}"/>
+        <mesh filename="package://robbie/mesh/waist top upper left.stl" scale="${M_SCALE} ${M_SCALE} ${M_SCALE}"/>
       </geometry>
           <xacro:cyan3 />
@@ -79,5 +79,5 @@
    <visual>
       <geometry>
-        <mesh filename="package://robbie/meshes/waist top upper right.stl" scale="${M_SCALE} ${M_SCALE} ${M_SCALE}"/>
+        <mesh filename="package://robbie/mesh/waist top upper right.stl" scale="${M_SCALE} ${M_SCALE} ${M_SCALE}"/>
       </geometry>
           <xacro:cyan3 />
@@ -89,5 +89,5 @@
    <visual>
       <geometry>
-        <mesh filename="package://robbie/meshes/gear_box.stl" scale="${M_SCALE} ${M_SCALE} ${M_SCALE}"/>
+        <mesh filename="package://robbie/mesh/gear_box.stl" scale="${M_SCALE} ${M_SCALE} ${M_SCALE}"/>
       </geometry>
        <material name="OffWhite">
@@ -100,5 +100,5 @@
    <visual>
       <geometry>
-        <mesh filename="package://robbie/meshes/shoulder_pan_gear.stl" scale="${M_SCALE} ${M_SCALE} ${M_SCALE}"/>
+        <mesh filename="package://robbie/mesh/shoulder_pan_gear.stl" scale="${M_SCALE} ${M_SCALE} ${M_SCALE}"/>
       </geometry>
        <xacro:yellow2 />
@@ -109,5 +109,5 @@
    <visual>
       <geometry>
-        <mesh filename="package://robbie/meshes/elbow_pivot.stl" scale="${M_SCALE} ${M_SCALE} ${M_SCALE}"/>
+        <mesh filename="package://robbie/mesh/elbow_pivot.stl" scale="${M_SCALE} ${M_SCALE} ${M_SCALE}"/>
       </geometry>
        <xacro:yellow2 />
@@ -118,5 +118,5 @@
    <visual>
       <geometry>
-        <mesh filename="package://robbie/meshes/shoulder_lift_bracket.stl" scale="${M_SCALE} ${M_SCALE} ${M_SCALE}"/>
+        <mesh filename="package://robbie/mesh/shoulder_lift_bracket.stl" scale="${M_SCALE} ${M_SCALE} ${M_SCALE}"/>
       </geometry>
        <xacro:yellow2 />
@@ -127,5 +127,5 @@
    <visual>
       <geometry>
-        <mesh filename="package://robbie/meshes/gear_box.stl" scale="${M_SCALE} ${M_SCALE} ${M_SCALE}"/>
+        <mesh filename="package://robbie/mesh/gear_box.stl" scale="${M_SCALE} ${M_SCALE} ${M_SCALE}"/>
       </geometry>
        <material name="OffWhite">
@@ -138,5 +138,5 @@
    <visual>
       <geometry>
-        <mesh filename="package://robbie/meshes/arm_top_left.stl" scale="${M_SCALE} ${M_SCALE} ${M_SCALE}"/>
+        <mesh filename="package://robbie/mesh/arm_top_left.stl" scale="${M_SCALE} ${M_SCALE} ${M_SCALE}"/>
       </geometry>
        <xacro:yellow2 />
@@ -147,5 +147,5 @@
    <visual>
       <geometry>
-        <mesh filename="package://robbie/meshes/right_arm _middle front.stl" scale="${M_SCALE} ${M_SCALE} ${M_SCALE}"/>
+        <mesh filename="package://robbie/mesh/right_arm _middle front.stl" scale="${M_SCALE} ${M_SCALE} ${M_SCALE}"/>
       </geometry>
        <xacro:blue1 />
@@ -156,5 +156,5 @@
    <visual>
       <geometry>
-        <mesh filename="package://robbie/meshes/elbow_plug.stl" scale="${M_SCALE} ${M_SCALE} ${M_SCALE}"/>
+        <mesh filename="package://robbie/mesh/elbow_plug.stl" scale="${M_SCALE} ${M_SCALE} ${M_SCALE}"/>
       </geometry>
        <xacro:yellow2 />
@@ -165,5 +165,5 @@
    <visual>
       <geometry>
-        <mesh filename="package://robbie/meshes/right_arm lower top.stl" scale="${M_SCALE} ${M_SCALE} ${M_SCALE}"/>
+        <mesh filename="package://robbie/mesh/right_arm lower top.stl" scale="${M_SCALE} ${M_SCALE} ${M_SCALE}"/>
       </geometry>
        <xacro:blue1 />
@@ -174,5 +174,5 @@
    <visual>
       <geometry>
-        <mesh filename="package://robbie/meshes/gear_box.stl" scale="${M_SCALE} ${M_SCALE} ${M_SCALE}"/>
+        <mesh filename="package://robbie/mesh/gear_box.stl" scale="${M_SCALE} ${M_SCALE} ${M_SCALE}"/>
       </geometry>
        <xacro:yellow2 />
@@ -183,5 +183,5 @@
    <visual>
       <geometry>
-        <mesh filename="package://robbie/meshes/elbow_pivot.stl" scale="${M_SCALE} ${M_SCALE} ${M_SCALE}"/>
+        <mesh filename="package://robbie/mesh/elbow_pivot.stl" scale="${M_SCALE} ${M_SCALE} ${M_SCALE}"/>
       </geometry>
        <xacro:yellow2 />
@@ -192,5 +192,5 @@
     <visual>
       <geometry>
-        <mesh filename="package://robbie/meshes/fore_arm.stl" scale="${M_SCALE} ${M_SCALE} ${M_SCALE}"/>
+        <mesh filename="package://robbie/mesh/fore_arm.stl" scale="${M_SCALE} ${M_SCALE} ${M_SCALE}"/>
       </geometry>
         <xacro:yellow2 />
@@ -218,5 +218,5 @@
    <visual>
       <geometry>
-        <mesh filename="package://robbie/meshes/gear_box.stl" scale="${M_SCALE} ${M_SCALE} ${M_SCALE}"/>
+        <mesh filename="package://robbie/mesh/gear_box.stl" scale="${M_SCALE} ${M_SCALE} ${M_SCALE}"/>
       </geometry>
        <material name="green">
@@ -229,5 +229,5 @@
    <visual>
       <geometry>
-        <mesh filename="package://robbie/meshes/shoulder_pan_gear.stl" scale="${M_SCALE} ${M_SCALE} ${M_SCALE}"/>
+        <mesh filename="package://robbie/mesh/shoulder_pan_gear.stl" scale="${M_SCALE} ${M_SCALE} ${M_SCALE}"/>
       </geometry>
        <xacro:yellow2 />
@@ -238,5 +238,5 @@
    <visual>
       <geometry>
-        <mesh filename="package://robbie/meshes/elbow_pivot.stl" scale="${M_SCALE} ${M_SCALE} ${M_SCALE}"/>
+        <mesh filename="package://robbie/mesh/elbow_pivot.stl" scale="${M_SCALE} ${M_SCALE} ${M_SCALE}"/>
       </geometry>
        <xacro:yellow2 />
@@ -247,5 +247,5 @@
    <visual>
       <geometry>
-        <mesh filename="package://robbie/meshes/shoulder_lift_bracket_left.stl" scale="${M_SCALE} ${M_SCALE} ${M_SCALE}"/>
+        <mesh filename="package://robbie/mesh/shoulder_lift_bracket_left.stl" scale="${M_SCALE} ${M_SCALE} ${M_SCALE}"/>
       </geometry>
        <xacro:yellow2 />
@@ -256,5 +256,5 @@
    <visual>
       <geometry>
-        <mesh filename="package://robbie/meshes/gear_box.stl" scale="${M_SCALE} ${M_SCALE} ${M_SCALE}"/>
+        <mesh filename="package://robbie/mesh/gear_box.stl" scale="${M_SCALE} ${M_SCALE} ${M_SCALE}"/>
       </geometry>
        <material name="OffWhite">
@@ -267,5 +267,5 @@
    <visual>
       <geometry>
-        <mesh filename="package://robbie/meshes/left_top_shoulder.stl" scale="${M_SCALE} ${M_SCALE} ${M_SCALE}"/>
+        <mesh filename="package://robbie/mesh/left_top_shoulder.stl" scale="${M_SCALE} ${M_SCALE} ${M_SCALE}"/>
       </geometry>
        <xacro:yellow2 />
@@ -276,5 +276,5 @@
    <visual>
       <geometry>
-        <mesh filename="package://robbie/meshes/left_mid_front.stl" scale="${M_SCALE} ${M_SCALE} ${M_SCALE}"/>
+        <mesh filename="package://robbie/mesh/left_mid_front.stl" scale="${M_SCALE} ${M_SCALE} ${M_SCALE}"/>
       </geometry>
        <xacro:blue1 />
@@ -285,5 +285,5 @@
    <visual>
       <geometry>
-        <mesh filename="package://robbie/meshes/elbow_plug.stl" scale="${M_SCALE} ${M_SCALE} ${M_SCALE}"/>
+        <mesh filename="package://robbie/mesh/elbow_plug.stl" scale="${M_SCALE} ${M_SCALE} ${M_SCALE}"/>
       </geometry>
        <xacro:yellow2 />
@@ -294,5 +294,5 @@
    <visual>
       <geometry>
-        <mesh filename="package://robbie/meshes/right_arm lower top.stl" scale="${M_SCALE} ${M_SCALE} ${M_SCALE}"/>
+        <mesh filename="package://robbie/mesh/right_arm lower top.stl" scale="${M_SCALE} ${M_SCALE} ${M_SCALE}"/>
       </geometry>
        <xacro:blue1 />
@@ -303,5 +303,5 @@
    <visual>
       <geometry>
-        <mesh filename="package://robbie/meshes/gear_box.stl" scale="${M_SCALE} ${M_SCALE} ${M_SCALE}"/>
+        <mesh filename="package://robbie/mesh/gear_box.stl" scale="${M_SCALE} ${M_SCALE} ${M_SCALE}"/>
       </geometry>
        <xacro:yellow2 />
@@ -312,5 +312,5 @@
    <visual>
       <geometry>
-        <mesh filename="package://robbie/meshes/elbow_pivot.stl" scale="${M_SCALE} ${M_SCALE} ${M_SCALE}"/>
+        <mesh filename="package://robbie/mesh/elbow_pivot.stl" scale="${M_SCALE} ${M_SCALE} ${M_SCALE}"/>
       </geometry>
        <xacro:yellow2 />
@@ -321,5 +321,5 @@
     <visual>
       <geometry>
-        <mesh filename="package://robbie/meshes/fore_arm.stl" scale="${M_SCALE} ${M_SCALE} ${M_SCALE}"/>
+        <mesh filename="package://robbie/mesh/fore_arm.stl" scale="${M_SCALE} ${M_SCALE} ${M_SCALE}"/>
       </geometry>
         <xacro:yellow2 />
@@ -358,5 +358,5 @@
    <visual>
       <geometry>
-        <mesh filename="package://robbie/meshes/head.stl" scale="${M_SCALE} ${M_SCALE} ${M_SCALE}"/>
+        <mesh filename="package://robbie/mesh/head.stl" scale="${M_SCALE} ${M_SCALE} ${M_SCALE}"/>
       </geometry>
          <material name="grey1">
@@ -375,4 +375,48 @@
       </inertial>
     </link>
+   <link name="kinect_link">
+      <inertial>
+        <mass value="1.0" />
+        <origin xyz="0 0 0" />
+        <inertia ixx="1.0" ixy="0.0" ixz="0.0"
+                 iyy="1.0" iyz="0.0"
+                 izz="1.0" />
+      </inertial>
+      <visual>
+        <origin xyz=" 0 0 0 " rpy="0 0 0" />
+        <geometry>
+          <mesh filename="package://robbie/meshes/kinect.stl" scale="${M_SCALE} ${M_SCALE} ${M_SCALE}"/>
+        </geometry>
+        <xacro:ax12_color />
+      </visual>
+      <collision>
+        <origin xyz="0 0 0" rpy="0 0 0" />
+        <geometry>
+          <mesh filename="package://robbie/meshes/kinect.stl" scale="${M_SCALE} ${M_SCALE} ${M_SCALE}"/>
+          </geometry>
+      </collision>
+    </link>
+  <link name="head_cam_link">
+      <inertial>
+        <mass value="1.0" />
+        <origin xyz="0 0 0" />
+        <inertia ixx="1.0" ixy="0.0" ixz="0.0"
+                 iyy="1.0" iyz="0.0"
+                 izz="1.0" />
+      </inertial>
+      <visual>
+        <origin xyz=" 0 0 0 " rpy="0 0 0" />
+        <geometry>
+          <mesh filename="package://robbie/meshes/kinect.stl" scale="${M_SCALE} ${M_SCALE} ${M_SCALE}"/>
+        </geometry>
+          <xacro:grey3 />
+      </visual>
+      <collision>
+        <origin xyz="0 0 0" rpy="0 0 0" />
+        <geometry>
+          <mesh filename="package://robbie/meshes/kinect.stl" scale="${M_SCALE} ${M_SCALE} ${M_SCALE}"/>
+          </geometry>
+      </collision>
+    </link>
 <!-- =================== Joint Definitions ==================== -->
   <joint name="base_link_joint" type="fixed">
@@ -432,5 +476,5 @@
     	<origin xyz="0.0 0.03 0.01" rpy="0 0 0" />
 	</joint>
-<!--###########################3right arm############################################3-->
+<!--########################### right arm############################################3-->
   <joint name="right_arm_pan_joint" type="revolute">
     <parent link="upper_torso"/>
@@ -568,5 +612,5 @@
     	<origin xyz="-0.025 0.05 0.105" rpy="0 0 0" />
 	</joint>
-  <joint name="left_arm_pan_joint" type="revolute">
+  <joint name="left_arm_pan_joint" type="fixed"> <!--revolute-->
     <parent link="upper_torso"/>
     <child link="left_shoulder_pan"/>
@@ -575,5 +619,5 @@
    <limit lower="-1.57" upper="1.57" effort="10" velocity="0" />
   </joint>
-  <joint name="left_arm_tilt_joint" type="revolute">
+  <joint name="left_arm_tilt_joint" type="fixed"> <!--revolute-->
     <parent link="left_shoulder_gear"/>
     <child link="left_shoulder_tilt"/>
@@ -592,8 +636,8 @@
     	<origin xyz="0.03 0.005 -0.055" rpy="0 0 0" />
 	</joint>
-  <joint name="left_arm_lift_joint" type="revolute">
+  <joint name="left_arm_lift_joint" type="fixed"> <!--revolute-->
     <parent link="left_shoulder_lift"/>
     <child link="left_shoulder_lift2"/>
-    <origin xyz="-0.025 -0.03 0.035" rpy="0 -1.57 0" />
+    <origin xyz="-0.025 -0.03 0.035" rpy="0 0 0" /><!--rpy="0 -1.57 0"-->
     <axis xyz="0 1 0" />
    <limit lower="-1.57" upper="1.9" effort="10" velocity="0" />
@@ -604,5 +648,5 @@
     	<origin xyz="-0.067 0.07 -0.093" rpy="0 0 0" />
 	</joint>
-  <joint name="left_arm_rotate_joint" type="revolute">
+  <joint name="left_arm_rotate_joint" type="fixed"> <!--revolute-->
     	<parent link="left_shoulder_mid" />
     	<child link="left_shoulder_lower" />
@@ -621,5 +665,5 @@
     	<origin xyz="-0.09 0.08 -0.13" rpy="0 0 0" />
 	</joint>
-  <joint name="left_arm_elbow_joint" type="revolute">
+  <joint name="left_arm_elbow_joint" type="fixed"> <!--revolute-->
     <parent link="left_elbow_gearbox"/>
     <child link="left_elbow"/>
@@ -639,5 +683,5 @@
     	<origin xyz="-0.21 0.0 0.0" rpy="0 0 1.57" /><!--now-->
 	</joint>
-  <joint name="left_arm_wrist_pan_joint" type="revolute">
+  <joint name="left_arm_wrist_pan_joint" type="fixed"> <!--revolute-->
     	<parent link="left_wrist_pan_servo" />
     	<child link="left_wrist_pan_servo_bracket_f3" />
@@ -654,5 +698,5 @@
 	</joint>
 <!--wrist_tilt_joint-->
-  <joint name="left_arm_wrist_tilt_joint" type="revolute">
+  <joint name="left_arm_wrist_tilt_joint" type="fixed"> <!--revolute-->
     	<parent link="left_wrist_tilt_servo" />
     	<child link="left_wrist_tilt_bracket_f2" />
@@ -673,5 +717,5 @@
 	</joint>
   <!-- left gripper_joint-->
-   <joint name="left_arm_gripper_joint" type="revolute">
+   <joint name="left_arm_gripper_joint" type="fixed"> <!--revolute-->
     	<parent link="left_gripper_servo" />
     	<child link="left_gripper_bracket_f2" />
@@ -745,4 +789,98 @@
     	<origin xyz="-0.02 -0.097 -0.45" rpy="0 0 0" />
 	</joint>
+  <joint name="kinect_joint" type="fixed">
+    	<parent link="base_link" />
+    	<child link="kinect_link" />
+    	<origin xyz="0.2 0 0.26" rpy="0 0 0" />
+	</joint>
+  <joint name="kinect_depth_joint" type="fixed">
+      <origin xyz="0 0.018 0" rpy="0 0 0" />
+      <parent link="kinect_link" />
+      <child link="kinect_depth_frame" />
+    </joint>
+    <link name="kinect_depth_frame">
+      <inertial>
+        <mass value="0.0001" />
+        <origin xyz="0 0 0" />
+        <inertia ixx="0.0001" ixy="0.0" ixz="0.0"
+                 iyy="0.0001" iyz="0.0"
+                 izz="0.0001" />
+      </inertial>
+    </link>
+    <joint name="kinect_depth_optical_joint" type="fixed">
+      <origin xyz="0 0 0" rpy="${-M_PI/2} 0 ${-M_PI/2}" />
+      <parent link="kinect_link" />
+      <child link="kinect_depth_optical_frame" />
+    </joint>
+    <link name="kinect_depth_optical_frame">
+      <inertial>
+        <mass value="0.0001" />
+        <origin xyz="0 0 0" />
+        <inertia ixx="0.0001" ixy="0.0" ixz="0.0"
+                 iyy="0.0001" iyz="0.0"
+                 izz="0.0001" />
+      </inertial>
+    </link>
+    <joint name="kinect_rgb_optical_joint" type="fixed">
+      <origin xyz="0 0 0" rpy="${-M_PI/2} 0 ${-M_PI/2}" />
+      <parent link="kinect_depth_optical_frame" />
+      <child link="kinect_rgb_optical_frame" />
+    </joint>
+    <link name="kinect_rgb_optical_frame">
+      <inertial>
+        <mass value="0.001" />
+        <origin xyz="0 0 0" />
+        <inertia ixx="0.0001" ixy="0.0" ixz="0.0"
+                 iyy="0.0001" iyz="0.0"
+                 izz="0.0001" />
+      </inertial>
+    </link>
+  <joint name="head_cam_joint" type="fixed">
+    	<parent link="head_link" />
+    	<child link="head_cam_link" />
+    	<origin xyz="0.15 0.1 0.58" rpy="0 0 0" />
+	</joint>
+  <joint name="head_cam_depth_joint" type="fixed">
+      <origin xyz="0 0.018 0" rpy="0 0 0" />
+      <parent link="head_cam_link" />
+      <child link="head_cam_depth_frame" />
+    </joint>
+    <link name="head_cam_depth_frame">
+      <inertial>
+        <mass value="0.0001" />
+        <origin xyz="0 0 0" />
+        <inertia ixx="0.0001" ixy="0.0" ixz="0.0"
+                 iyy="0.0001" iyz="0.0"
+                 izz="0.0001" />
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