Commit message: various updates

File: urdf/robbie7.xacro (robot description, xacro)
@@ -32,5 +32,5 @@
    <visual>
       <geometry>
-        <mesh filename="package://robbie/mesh/upper_torso2.stl" scale="${M_SCALE} ${M_SCALE} ${M_SCALE}"/>
+        <mesh filename="package://robbie/meshes/upper_torso2.stl" scale="${M_SCALE} ${M_SCALE} ${M_SCALE}"/>
       </geometry>
          <material name="green">
@@ -43,5 +43,5 @@
    <visual>
       <geometry>
-        <mesh filename="package://robbie/mesh/bottom torso.stl" scale="${M_SCALE} ${M_SCALE} ${M_SCALE}"/>
+        <mesh filename="package://robbie/meshes/bottom torso.stl" scale="${M_SCALE} ${M_SCALE} ${M_SCALE}"/>
       </geometry>
           <xacro:cyan3 />
@@ -52,5 +52,5 @@
    <visual>
       <geometry>
-        <mesh filename="package://robbie/mesh/waist top lower left.stl" scale="${M_SCALE} ${M_SCALE} ${M_SCALE}"/>
+        <mesh filename="package://robbie/meshes/waist top lower left.stl" scale="${M_SCALE} ${M_SCALE} ${M_SCALE}"/>
       </geometry>
           <xacro:cyan3 />
@@ -61,5 +61,5 @@
    <visual>
       <geometry>
-        <mesh filename="package://robbie/mesh/waist top lower right.stl" scale="${M_SCALE} ${M_SCALE} ${M_SCALE}"/>
+        <mesh filename="package://robbie/meshes/waist top lower right.stl" scale="${M_SCALE} ${M_SCALE} ${M_SCALE}"/>
       </geometry>
           <xacro:cyan3 />
@@ -70,5 +70,5 @@
    <visual>
       <geometry>
-        <mesh filename="package://robbie/mesh/waist top upper left.stl" scale="${M_SCALE} ${M_SCALE} ${M_SCALE}"/>
+        <mesh filename="package://robbie/meshes/waist top upper left.stl" scale="${M_SCALE} ${M_SCALE} ${M_SCALE}"/>
       </geometry>
           <xacro:cyan3 />
@@ -79,5 +79,5 @@
    <visual>
       <geometry>
-        <mesh filename="package://robbie/mesh/waist top upper right.stl" scale="${M_SCALE} ${M_SCALE} ${M_SCALE}"/>
+        <mesh filename="package://robbie/meshes/waist top upper right.stl" scale="${M_SCALE} ${M_SCALE} ${M_SCALE}"/>
       </geometry>
           <xacro:cyan3 />
@@ -89,10 +89,10 @@
    <visual>
       <geometry>
-        <mesh filename="package://robbie/mesh/gear_box.stl" scale="${M_SCALE} ${M_SCALE} ${M_SCALE}"/>
+        <mesh filename="package://robbie/meshes/gear_box.stl" scale="${M_SCALE} ${M_SCALE} ${M_SCALE}"/>
       </geometry>
        <material name="OffWhite">
        <color rgba="0.8 0.8 0.8 0.9"/>
        </material>
-      <origin rpy="-1.57 0 1.57" xyz="0 0 0"/>
+      <origin rpy="${-M_PI/2} 0 1.57" xyz="0 0 0"/>
     </visual>
   </link>
@@ -100,8 +100,8 @@
    <visual>
       <geometry>
-        <mesh filename="package://robbie/mesh/shoulder_pan_gear.stl" scale="${M_SCALE} ${M_SCALE} ${M_SCALE}"/>
-      </geometry>
-       <xacro:yellow2 />
-      <origin rpy="0 0 -1.57" xyz="-0.05 0.05 0.0"/>
+        <mesh filename="package://robbie/meshes/shoulder_pan_gear.stl" scale="${M_SCALE} ${M_SCALE} ${M_SCALE}"/>
+      </geometry>
+       <xacro:yellow2 />
+      <origin rpy="0 0 ${-M_PI/2}" xyz="-0.05 0.05 0.0"/>
     </visual>
   </link>
@@ -109,8 +109,8 @@
    <visual>
       <geometry>
-        <mesh filename="package://robbie/mesh/elbow_pivot.stl" scale="${M_SCALE} ${M_SCALE} ${M_SCALE}"/>
-      </geometry>
-       <xacro:yellow2 />
-      <origin rpy="0 0 1.57" xyz="-0.045 0.02 -0.03"/>
+        <mesh filename="package://robbie/meshes/elbow_pivot.stl" scale="${M_SCALE} ${M_SCALE} ${M_SCALE}"/>
+      </geometry>
+       <xacro:yellow2 />
+      <origin rpy="0 0 ${M_PI/2}" xyz="-0.045 0.02 -0.03"/>
     </visual>
   </link>
@@ -118,8 +118,8 @@
    <visual>
       <geometry>
-        <mesh filename="package://robbie/mesh/shoulder_lift_bracket.stl" scale="${M_SCALE} ${M_SCALE} ${M_SCALE}"/>
-      </geometry>
-       <xacro:yellow2 />
-      <origin rpy="0 1.57 1.57" xyz="0 0 0"/>
+        <mesh filename="package://robbie/meshes/shoulder_lift_bracket.stl" scale="${M_SCALE} ${M_SCALE} ${M_SCALE}"/>
+      </geometry>
+       <xacro:yellow2 />
+      <origin rpy="0 ${M_PI/2} ${M_PI/2}" xyz="0 0 0"/>
     </visual>
   </link>
@@ -127,5 +127,5 @@
    <visual>
       <geometry>
-        <mesh filename="package://robbie/mesh/gear_box.stl" scale="${M_SCALE} ${M_SCALE} ${M_SCALE}"/>
+        <mesh filename="package://robbie/meshes/gear_box.stl" scale="${M_SCALE} ${M_SCALE} ${M_SCALE}"/>
       </geometry>
        <material name="OffWhite">
@@ -138,5 +138,5 @@
    <visual>
       <geometry>
-        <mesh filename="package://robbie/mesh/arm_top_left.stl" scale="${M_SCALE} ${M_SCALE} ${M_SCALE}"/>
+        <mesh filename="package://robbie/meshes/arm_top_left.stl" scale="${M_SCALE} ${M_SCALE} ${M_SCALE}"/>
       </geometry>
        <xacro:yellow2 />
@@ -147,5 +147,5 @@
    <visual>
       <geometry>
-        <mesh filename="package://robbie/mesh/right_arm _middle front.stl" scale="${M_SCALE} ${M_SCALE} ${M_SCALE}"/>
+        <mesh filename="package://robbie/meshes/right_arm _middle front.stl" scale="${M_SCALE} ${M_SCALE} ${M_SCALE}"/>
       </geometry>
        <xacro:blue1 />
@@ -156,5 +156,5 @@
    <visual>
       <geometry>
-        <mesh filename="package://robbie/mesh/elbow_plug.stl" scale="${M_SCALE} ${M_SCALE} ${M_SCALE}"/>
+        <mesh filename="package://robbie/meshes/elbow_plug.stl" scale="${M_SCALE} ${M_SCALE} ${M_SCALE}"/>
       </geometry>
        <xacro:yellow2 />
@@ -165,5 +165,5 @@
    <visual>
       <geometry>
-        <mesh filename="package://robbie/mesh/right_arm lower top.stl" scale="${M_SCALE} ${M_SCALE} ${M_SCALE}"/>
+        <mesh filename="package://robbie/meshes/right_arm lower top.stl" scale="${M_SCALE} ${M_SCALE} ${M_SCALE}"/>
       </geometry>
        <xacro:blue1 />
@@ -174,8 +174,8 @@
    <visual>
       <geometry>
-        <mesh filename="package://robbie/mesh/gear_box.stl" scale="${M_SCALE} ${M_SCALE} ${M_SCALE}"/>
-      </geometry>
-       <xacro:yellow2 />
-      <origin rpy="1.57 0 0" xyz="0 0 0"/>
+        <mesh filename="package://robbie/meshes/gear_box.stl" scale="${M_SCALE} ${M_SCALE} ${M_SCALE}"/>
+      </geometry>
+       <xacro:yellow2 />
+      <origin rpy="1.57 0 3.14" xyz="0.06 -0.04 0"/>
     </visual>
   </link>
@@ -183,5 +183,5 @@
    <visual>
       <geometry>
-        <mesh filename="package://robbie/mesh/elbow_pivot.stl" scale="${M_SCALE} ${M_SCALE} ${M_SCALE}"/>
+        <mesh filename="package://robbie/meshes/elbow_pivot.stl" scale="${M_SCALE} ${M_SCALE} ${M_SCALE}"/>
       </geometry>
        <xacro:yellow2 />
@@ -192,5 +192,5 @@
     <visual>
       <geometry>
-        <mesh filename="package://robbie/mesh/fore_arm.stl" scale="${M_SCALE} ${M_SCALE} ${M_SCALE}"/>
+        <mesh filename="package://robbie/meshes/fore_arm.stl" scale="${M_SCALE} ${M_SCALE} ${M_SCALE}"/>
       </geometry>
         <xacro:yellow2 />
@@ -218,5 +218,5 @@
    <visual>
       <geometry>
-        <mesh filename="package://robbie/mesh/gear_box.stl" scale="${M_SCALE} ${M_SCALE} ${M_SCALE}"/>
+        <mesh filename="package://robbie/meshes/gear_box.stl" scale="${M_SCALE} ${M_SCALE} ${M_SCALE}"/>
       </geometry>
        <material name="green">
@@ -229,5 +229,5 @@
    <visual>
       <geometry>
-        <mesh filename="package://robbie/mesh/shoulder_pan_gear.stl" scale="${M_SCALE} ${M_SCALE} ${M_SCALE}"/>
+        <mesh filename="package://robbie/meshes/shoulder_pan_gear.stl" scale="${M_SCALE} ${M_SCALE} ${M_SCALE}"/>
       </geometry>
        <xacro:yellow2 />
@@ -238,5 +238,5 @@
    <visual>
       <geometry>
-        <mesh filename="package://robbie/mesh/elbow_pivot.stl" scale="${M_SCALE} ${M_SCALE} ${M_SCALE}"/>
+        <mesh filename="package://robbie/meshes/elbow_pivot.stl" scale="${M_SCALE} ${M_SCALE} ${M_SCALE}"/>
       </geometry>
        <xacro:yellow2 />
@@ -247,5 +247,5 @@
    <visual>
       <geometry>
-        <mesh filename="package://robbie/mesh/shoulder_lift_bracket_left.stl" scale="${M_SCALE} ${M_SCALE} ${M_SCALE}"/>
+        <mesh filename="package://robbie/meshes/shoulder_lift_bracket_left.stl" scale="${M_SCALE} ${M_SCALE} ${M_SCALE}"/>
       </geometry>
        <xacro:yellow2 />
@@ -256,5 +256,5 @@
    <visual>
       <geometry>
-        <mesh filename="package://robbie/mesh/gear_box.stl" scale="${M_SCALE} ${M_SCALE} ${M_SCALE}"/>
+        <mesh filename="package://robbie/meshes/gear_box.stl" scale="${M_SCALE} ${M_SCALE} ${M_SCALE}"/>
       </geometry>
        <material name="OffWhite">
@@ -267,5 +267,5 @@
    <visual>
       <geometry>
-        <mesh filename="package://robbie/mesh/left_top_shoulder.stl" scale="${M_SCALE} ${M_SCALE} ${M_SCALE}"/>
+        <mesh filename="package://robbie/meshes/left_top_shoulder.stl" scale="${M_SCALE} ${M_SCALE} ${M_SCALE}"/>
       </geometry>
        <xacro:yellow2 />
@@ -276,5 +276,5 @@
    <visual>
       <geometry>
-        <mesh filename="package://robbie/mesh/left_mid_front.stl" scale="${M_SCALE} ${M_SCALE} ${M_SCALE}"/>
+        <mesh filename="package://robbie/meshes/left_mid_front.stl" scale="${M_SCALE} ${M_SCALE} ${M_SCALE}"/>
       </geometry>
        <xacro:blue1 />
@@ -285,5 +285,5 @@
    <visual>
       <geometry>
-        <mesh filename="package://robbie/mesh/elbow_plug.stl" scale="${M_SCALE} ${M_SCALE} ${M_SCALE}"/>
+        <mesh filename="package://robbie/meshes/elbow_plug.stl" scale="${M_SCALE} ${M_SCALE} ${M_SCALE}"/>
       </geometry>
        <xacro:yellow2 />
@@ -294,5 +294,5 @@
    <visual>
       <geometry>
-        <mesh filename="package://robbie/mesh/right_arm lower top.stl" scale="${M_SCALE} ${M_SCALE} ${M_SCALE}"/>
+        <mesh filename="package://robbie/meshes/right_arm lower top.stl" scale="${M_SCALE} ${M_SCALE} ${M_SCALE}"/>
       </geometry>
        <xacro:blue1 />
@@ -303,8 +303,8 @@
    <visual>
       <geometry>
-        <mesh filename="package://robbie/mesh/gear_box.stl" scale="${M_SCALE} ${M_SCALE} ${M_SCALE}"/>
-      </geometry>
-       <xacro:yellow2 />
-      <origin rpy="1.57 0 0" xyz="0 0 0"/>
+        <mesh filename="package://robbie/meshes/gear_box.stl" scale="${M_SCALE} ${M_SCALE} ${M_SCALE}"/>
+      </geometry>
+       <xacro:yellow2 />
+      <origin rpy="1.57 0 3.14" xyz="0.06 -0.04 0"/>
     </visual>
   </link>
@@ -312,5 +312,5 @@
    <visual>
       <geometry>
-        <mesh filename="package://robbie/mesh/elbow_pivot.stl" scale="${M_SCALE} ${M_SCALE} ${M_SCALE}"/>
+        <mesh filename="package://robbie/meshes/elbow_pivot.stl" scale="${M_SCALE} ${M_SCALE} ${M_SCALE}"/>
       </geometry>
        <xacro:yellow2 />
@@ -321,5 +321,5 @@
     <visual>
       <geometry>
-        <mesh filename="package://robbie/mesh/fore_arm.stl" scale="${M_SCALE} ${M_SCALE} ${M_SCALE}"/>
+        <mesh filename="package://robbie/meshes/fore_arm.stl" scale="${M_SCALE} ${M_SCALE} ${M_SCALE}"/>
       </geometry>
         <xacro:yellow2 />
@@ -358,5 +358,5 @@
    <visual>
       <geometry>
-        <mesh filename="package://robbie/mesh/head.stl" scale="${M_SCALE} ${M_SCALE} ${M_SCALE}"/>
+        <mesh filename="package://robbie/meshes/head.stl" scale="${M_SCALE} ${M_SCALE} ${M_SCALE}"/>
       </geometry>
          <material name="grey1">
@@ -375,5 +375,5 @@
       </inertial>
     </link>
-   <link name="kinect_link">
+    <link name="kinect_link">
       <inertial>
         <mass value="1.0" />
@@ -476,5 +476,5 @@
     	<origin xyz="0.0 0.03 0.01" rpy="0 0 0" />
 	</joint>
-<!--########################### right arm############################################3-->
+<!--###########################right arm############################################3-->
   <joint name="right_arm_pan_joint" type="revolute">
     <parent link="upper_torso"/>
@@ -482,5 +482,5 @@
     <origin xyz="-0.05 0.05 0.0" rpy="0  0 0" />
     <axis xyz="0 0 1" />
-   <limit lower="-1.57" upper="1.57" effort="10" velocity="0" />
+   <limit lower="-0.80" upper="0.80" effort="10" velocity="0" />
   </joint>
   <joint name="right_shoulder_link" type="fixed">
@@ -494,10 +494,10 @@
     <origin xyz="-0.02 0.03 -0.03" rpy="0 0 0" />
     <axis xyz="1 0 0" />
-   <limit lower="-1.57" upper="1.57" effort="10" velocity="0" />
+   <limit lower="-0.82" upper="0" effort="10" velocity="0" />
   </joint>
   <joint name="right_shoulder_lift_bracket_link" type="fixed">
     	<parent link="right_shoulder_tilt" />
     	<child link="right_shoulder_bracket" />
-    	<origin xyz="0.09 -0.125 0.02" rpy="0 0 0" />
+    	<origin xyz="0.01 -0.145 0.02" rpy="0 0 0" />
 	</joint>
   <joint name="right_shoulder_lift_gearbox_link" type="fixed">
@@ -511,5 +511,5 @@
     <origin xyz="-0.025 -0.075 0.035" rpy="0 -1.57 0" />
     <axis xyz="0 1 0" />
-   <limit lower="-1.57" upper="1.9" effort="10" velocity="0" />
+   <limit lower="-1.1" upper="1.9" effort="10" velocity="0" />
   </joint>
   <joint name="right_shoulder_mid_link" type="fixed">
@@ -523,5 +523,5 @@
     	<origin xyz="-0.07 0.052 -0.131" rpy="0 0 0" />
         <axis xyz="0 0 1" />
-        <limit lower="-2.00" upper="1.57" effort="10" velocity="0" />
+        <limit lower="-1.57" upper="1.57" effort="10" velocity="0" />
 	</joint>
   <joint name="right_shoulder_elbow_link" type="fixed">
@@ -538,5 +538,5 @@
     <parent link="right_elbow_gearbox"/>
     <child link="right_elbow"/>
-    <origin xyz="0.02 -0.02 0.025" rpy="0 -1.57 0" />
+    <origin xyz="0.03 -0.02 0.025" rpy="0 -1.57 0" />
     <axis xyz="0 1 0" />
    <limit lower="-2.00" upper="0.57" effort="10" velocity="0" />
@@ -617,5 +617,5 @@
     <origin xyz="-0.04 0.22 0.0" rpy="0  0 0" />
     <axis xyz="0 0 1" />
-   <limit lower="-1.57" upper="1.57" effort="10" velocity="0" />
+   <limit lower="-0.80" upper="0.80" effort="10" velocity="0" />
   </joint>
   <joint name="left_arm_tilt_joint" type="fixed"> <!--revolute-->
@@ -624,10 +624,10 @@
     <origin xyz="0.02 -0.03 -0.03" rpy="0 0 0" />
     <axis xyz="1 0 0" />
-   <limit lower="-1.57" upper="1.57" effort="10" velocity="0" />
+   <limit lower="-0.82" upper="0.0" effort="10" velocity="0" />
   </joint>
   <joint name="left_shoulder_lift_bracket_link" type="fixed">
     	<parent link="left_shoulder_tilt" />
     	<child link="left_shoulder_bracket" />
-    	<origin xyz="0.08 0.125 0.02" rpy="0 0 0" />
+    	<origin xyz="0.0 0.145 0.02" rpy="0 0 0" />
 	</joint>
   <joint name="left_shoulder_lift_gearbox_link" type="fixed">
@@ -641,5 +641,5 @@
     <origin xyz="-0.025 -0.03 0.035" rpy="0 0 0" /><!--rpy="0 -1.57 0"-->
     <axis xyz="0 1 0" />
-   <limit lower="-1.57" upper="1.9" effort="10" velocity="0" />
+   <limit lower="-1.1" upper="1.9" effort="10" velocity="0" />
   </joint>
   <joint name="left_shoulder_mid_link" type="fixed">
@@ -668,5 +668,5 @@
     <parent link="left_elbow_gearbox"/>
     <child link="left_elbow"/>
-    <origin xyz="0.02 -0.02 0.025" rpy="0 -1.57 0" />
+    <origin xyz="0.03 -0.02 0.025" rpy="0 -1.57 0" />
     <axis xyz="0 1 0" />
    <limit lower="-2.0" upper="0.57" effort="10" velocity="0" />
@@ -681,5 +681,5 @@
     	<parent link="left_forearm_link" />
     	<child link="left_wrist_pan_servo" />
-    	<origin xyz="-0.21 0.0 0.0" rpy="0 0 1.57" /><!--now-->
+    	<origin xyz="-0.21 0.0 0.0" rpy="0 0 1.57" />
 	</joint>
   <joint name="left_arm_wrist_pan_joint" type="fixed"> <!--revolute-->
@@ -731,5 +731,5 @@
 	</joint>
   <joint name="left_arm_finger_link_r" type="fixed">
-    	<parent link="left_gripper_servo" />
+    	<parent link="left_gripper_bracket_f2" />
     	<child link="left_right_finger_link" />
     	<origin xyz="0 0.03 0.03" rpy="0 0 0" />
@@ -789,8 +789,8 @@
     	<origin xyz="-0.02 -0.097 -0.45" rpy="0 0 0" />
 	</joint>
-  <joint name="kinect_joint" type="fixed">
+   <joint name="kinect_joint" type="fixed">
     	<parent link="base_link" />
     	<child link="kinect_link" />
-    	<origin xyz="0.2 0 0.26" rpy="0 0 0" />
+    	<origin xyz="0.2 0 0.47" rpy="0 0 0" />
 	</joint>
   <joint name="kinect_depth_joint" type="fixed">
@@ -839,6 +839,6 @@
     	<parent link="head_link" />
     	<child link="head_cam_link" />
-    	<origin xyz="0.15 0.1 0.58" rpy="0 0 0" />
-	</joint>
+    	<origin xyz="0.15 0.1 0.58" rpy="0 0 0" /><!-- 0 -1.57 1.57-->
+  </joint>
   <joint name="head_cam_depth_joint" type="fixed">
       <origin xyz="0 0.018 0" rpy="0 0 0" />
@@ -856,5 +856,5 @@
     </link>
     <joint name="head_cam_depth_optical_joint" type="fixed">
-      <origin xyz="0 0 0" rpy="${-M_PI/2} 0 ${-M_PI/2}" />
+      <origin xyz="0 0 0" rpy="${-M_PI/2} 0 0" />
       <parent link="head_cam_link" />
       <child link="head_cam_depth_optical_frame" />
@@ -870,5 +870,5 @@
     </link>
     <joint name="head_cam_rgb_optical_joint" type="fixed">
-      <origin xyz="0 0 0" rpy="${-M_PI/2} 0 ${-M_PI/2}" />
+      <origin xyz="0 0 0" rpy="0 ${M_PI/2} 0 " />
       <parent link="head_cam_depth_optical_frame" />
       <child link="head_cam_rgb_optical_frame" />
